File: OctoWatchScheme.brd (EAGLE design)
At the start: 35 x 34 mm, 23 parts, among them IC1 TP4056, IC2 DS1302, J1 0475900001, Y2 32.768kHz

Commit message: Pushing Scheme
Parts:
- moved R1 18.2 mm to (46.6, 45.1)
- moved C2 2.00 mm to (61.9, 61.0)
- moved U$2 0.50 mm to (60.5, 86.4)
- moved C5 0.30 mm to (69.4, 33.9), turned to 0 degrees
- moved C3 0.13 mm to (69.5, 36.5), turned to 180 degrees
Routing:
- net GND: track 32.2 -> 72.6 mm, vias 2 -> 5
- net N$13: track 6.01 -> 14.9 mm, vias 0 -> 1
- net N$29: track 0.00 -> 2.78 mm
- net N$15: track 22.4 -> 20.5 mm
- net N$25: track 10.5 -> 11.4 mm
- net N$8: track 18.5 -> 18.0 mm
- net N$23: track 8.72 -> 9.22 mm
