File: SCHEME/OctoWatchScheme.brd (EAGLE design)
At the start: 35 x 34 mm, 24 parts, among them IC1 TP4056, IC2 DS1302, J1 0475900001, Y2 32.768kHz

Commit message: GerBer Added
Routing:
- net N$7: track 29.3 -> 32.0 mm
- net N$17: track 37.7 -> 39.8 mm
- net N$8: track 18.2 -> 19.6 mm
- net N$13: track 16.9 -> 18.0 mm
- net N$4: track 15.9 -> 16.9 mm
- net BATT+: track 58.7 -> 59.4 mm

Commit message: working...
Connections:
- removed net N$16: IC2.I/O, U$2.P$9
- removed net N$21: U$2.P$12
- removed net N$24: R3.2, U$2.P$7
- removed net N$30: U$2.P$11, U$3.P$1
- new net N$20: U$2.P$12, U$3.P$1
- net BATT+: no longer R1.2, R2.2, R3.1
- net GND: now also R1.2, R2.2, R3.2, U$4.P$2
- net N$14: now also IC2.-RST, R3.1, U$2.P$7; no longer U$4.P$2
- net N$17: now also IC2.I/O, U$2.P$9; no longer IC2.-RST
- net N$23: now also IC2.SCLK
Routing:
- net N$17: track 39.8 -> 0.00 mm, vias 1 -> 0
- net N$30: track 29.3 -> 0.00 mm
- net N$16: track 28.4 -> 0.00 mm, vias 2 -> 0
- net GND: track 130.5 -> 109.3 mm
- net N$6: track 20.8 -> 0.00 mm, vias 1 -> 0
- net N$24: track 15.3 -> 0.00 mm, vias 1 -> 0
- net N$12: track 13.0 -> 0.00 mm, vias 1 -> 0
- net BATT+: track 59.4 -> 58.3 mm

Commit message: Adding new package
Parts:
- R7: device rcl:R1206 -> rcl:R0805
- U$2: device OctoWatch:STC15F204AE -> OctoWatch:STC15F204AE2
- moved U$2 22.9 mm to (50.7, 58.1)
- moved IC2 0.50 mm to (34.1, 49.3)
- moved Y2 0.50 mm to (32.9, 54.5)
- moved U$3 0.35 mm to (21.5, 31.8)
- moved U$4 0.35 mm to (71.8, 27.2)
Routing:
- net GND: track 109.3 -> 175.1 mm, vias 1 -> 0
- net N$14: track 0.00 -> 60.3 mm, vias 0 -> 2
- net N$17: track 0.00 -> 51.0 mm
- net N$20: track 0.00 -> 47.1 mm
- net N$6: track 0.00 -> 24.8 mm
- net N$23: track 7.14 -> 29.9 mm, vias 0 -> 1
- net N$7: track 32.0 -> 10.8 mm, vias 1 -> 0
- net N$19: track 45.1 -> 24.2 mm, vias 2 -> 0
- net N$10: track 22.7 -> 2.53 mm
- net N$18: track 22.3 -> 36.3 mm
- net BATT+: track 58.3 -> 44.9 mm
- net N$32: track 38.4 -> 50.2 mm, vias 2 -> 3
- net N$12: track 0.00 -> 11.0 mm
- net N$8: track 19.6 -> 13.2 mm
- net N$3: track 20.2 -> 16.2 mm
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