File: SCHEME/OctoWatchScheme2.brd (EAGLE design)
At the start: 35 x 34 mm, 23 parts, among them IC1 TP4056, IC2 DS1302, J1 0475900001

Commit message: adding 2nd ver
Parts:
- removed LED1, LED2: LG_T679-E1F1-1, led:PLCC2
- removed Y1: (no value), SparkFun-Clocks:CRYSTAL-SMD-2X6-CYL
- added BATT+: LSP13, solpad:LSP13
- added LED3, LED4: (no value), adafruit:CHIPLED_0603
- added Y2: 32.768kHz, SparkFun-Clocks:CRYSTAL-PTH-2X6-CYL
- R7: device rcl:R1206 -> adafruit:R0805
- moved BATT- 92.3 mm to (35.4, 42.1), turned to 90 degrees
- moved R1 77.6 mm to (16.5, 41.0)
- moved R6 75.9 mm to (18.6, 26.4)
- moved C5 74.5 mm to (29.0, 19.9)
- moved R5 72.2 mm to (18.7, 24.4)
- moved C4 68.6 mm to (29.1, 23.1)
- moved C3 64.0 mm to (29.2, 26.2), turned to 180 degrees
- moved R4 61.9 mm to (8.95, 20.2), turned to 90 degrees
- moved U$2 56.4 mm to (27.3, 80.4), turned to 90 degrees
- moved R7 52.1 mm to (12.1, 19.7), turned to 90 degrees
- moved C2 47.7 mm to (17.1, 47.8)
- moved C1 44.7 mm to (17.1, 49.6)
- moved IC1 42.9 mm to (11.5, 24.6)
- moved R3 39.8 mm to (16.4, 45.4)
- moved R2 37.6 mm to (16.4, 43.2)
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Connections:
- removed net AGND: BATT-.MP, C3.1, C4.2, C5.2, IC1.1, IC1.3, IC2.GND, J1.SH1, J1.SH2, J1.SH3, J1.SH4, J1.SH5, R4.1, R7.1, U$2.P$10, U$3.P$2
- removed net N$16: IC2.I/O, U$2.P$9
- removed net N$21: U$2.P$12
- removed net N$24: R3.2, U$2.P$7
- removed net N$25: R3.1, U$2.P$8
- removed net N$30: U$2.P$11, U$3.P$1
- removed net VCC: C3.2, C5.1, IC1.5, IC2.VCC1, IC2.VCC2, R2.2
- new net BATT+: C3.2, IC2.VCC1, IC2.VCC2, U$2.P$8
- new net GND: BATT-.MP, C1.2, C2.2, C3.1, C4.2, C5.2, IC1.1, IC1.3, IC2.GND, J1.5, J1.SH1, J1.SH2, J1.SH3, J1.SH4, J1.SH5, R1.2, R2.2, R3.2, R4.1, R7.1, U$2.P$10, U$3.P$2, U$3.P$3, U$3.P$4, U$4.P$2, U$4.P$3, U$4.P$4
- net N$13: now also Y2.1; no longer Y1.X1
- net N$14: now also IC2.-RST, R3.1, U$2.P$7; no longer C1.2, C2.2
- net N$15: now also Y2.2; no longer Y1.X2
- net N$17: now also IC2.I/O, U$2.P$9; no longer IC2.-RST
- net N$18: now also BATT+.MP, C5.1, IC1.5; no longer R1.2
- net N$20: now also U$2.P$12, U$3.P$1; no longer U$4.P$2
- net N$23: now also IC2.SCLK
- net N$27: now also LED4.C; no longer LED1.C
- net N$29: now also LED3.C; no longer LED2.C
- net N$32: now also LED3.A, LED4.A; no longer LED1.A, LED2.A
Routing:
- net GND: track 0.00 -> 153.8 mm, vias 0 -> 1
- net N$18: track 0.00 -> 52.2 mm, vias 0 -> 1
- net N$14: track 0.00 -> 51.4 mm, vias 0 -> 1
- net BATT+: track 0.00 -> 50.0 mm
- net N$11: track 0.00 -> 47.8 mm, vias 0 -> 3
- net N$32: track 0.00 -> 46.9 mm, vias 0 -> 2
- net N$6: track 0.00 -> 39.8 mm
- net N$17: track 0.00 -> 34.9 mm, vias 0 -> 1
- net N$23: track 0.00 -> 27.0 mm, vias 0 -> 1
- net N$20: track 0.00 -> 26.1 mm
- net N$12: track 0.00 -> 20.9 mm
- net N$1: track 0.00 -> 19.0 mm
- net N$8: track 0.00 -> 16.2 mm
- net N$3: track 26.7 -> 10.7 mm, vias 2 -> 0
- net N$7: track 0.00 -> 15.6 mm
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Other:
- outline, holes or cut-outs redrawn
