File: SCHEME/OctoWatchScheme2.sch (EAGLE design)
At the start: 23 parts, among them IC1 TP4056, IC2 DS1302, J1 0475900001, Y2 32.768kHz

Commit message: adding 2nd ver
Parts:
- added BATT+: LSP13, solpad:LSP13
- R7: device rcl:R-US_R1206 -> adafruit:R-US_R0805
Connections:
- removed net N$16: IC2.I/O, U$2.P0.1
- removed net N$21: U$2.P3.1
- removed net N$24: R3.2, U$2.RST
- removed net N$25: R3.1, U$2.VCC
- removed net N$30: U$2.INT4, U$3.SIGNAL
- removed net VCC: BATT-.MP, C3.2, C5.1, IC1.BAT, IC2.VCC1, IC2.VCC2, R2.2
- new net BATT+: C3.2, IC2.VCC1, IC2.VCC2, U$2.VCC
- new net N$20: U$2.P3.1, U$3.SIGNAL
- net GND: now also BATT-.MP, J1.GND, R1.2, R2.2, R3.2, U$3.P$1, U$3.P$2, U$4.GND, U$4.P$1, U$4.P$2
- net N$14: now also IC2.-RST, R3.1, U$2.RST; no longer U$4.GND
- net N$17: now also IC2.I/O, U$2.P0.1; no longer IC2.-RST
- net N$18: now also BATT+.MP, C5.1, IC1.BAT; no longer R1.2
- net N$23: now also IC2.SCLK
Other:
- moved on the sheet: BATT-, IC2, R1, R2, R3, U$3, U$4
