File: SCHEME/OctoWatchSchemePackage2NoWire.brd (EAGLE design)
At the start: 35 x 34 mm, 24 parts, among them IC1 TP4056, IC2 DS1302, J1 0475900001, Y2 32.768kHz

Commit message: Finalizing...
Parts:
- removed LED3, LED4: (no value), adafruit:CHIPLED_0603
- removed U$2: (no value), OctoWatch:STC15F204AE2
- added D1: SMD-LED-CLEAR-BLUE(0603), SMD-LED-CLEAR-BLUE_0603_:LED-0603
- added D2: LED-SMD-RED-DIFFUSED(0603), LED-SMD-RED-DIFFUSED_0603_:LED-0603
- added U$5: (no value), OctoWatch:STC15F204AE
- C1, C2: value 22pF -> CL21C220JBANNNC; device SparkFun-Capacitors:0402-TIGHT -> CL21C220JBANNNC:CAPC2012X140N
- C3: value 0.1uF -> CL21B104KCFNNNE; device SparkFun-Capacitors:0402 -> CL21B104KCFNNNE:CAPC2012X140N
- C4, C5: device rcl:C0805 -> GRT188R61E106ME13D:CAPC1608X100N
- R1, R2, R3: value 10k -> ERA3AEB103V; device SparkFun-Resistors:0603 -> ERA3AEB103V:RES_ERA3AEB103V
- R4: device rcl:R0402 -> AC1206FR-073K9L:RESC3116X65N
- R5, R6: device rcl:R0402 -> ERJ-PB3B1001V:RESC1608X55N
- moved BATT- 17.8 mm to (62.2, 40.9), turned to 0 degrees
- moved BATT+ 12.0 mm to (62.1, 36.4), turned to 0 degrees
- moved R2 10.2 mm to (61.7, 51.5), turned to 270 degrees
- moved C1 9.22 mm to (42.3, 47.5), turned to 0 degrees
- moved R1 8.55 mm to (61.8, 47.5), turned to 90 degrees
- moved R4 7.04 mm to (35.4, 26.2), turned to 90 degrees
- moved R3 4.32 mm to (55.6, 32.3), turned to 180 degrees
- moved C2 4.19 mm to (42.2, 51.2), turned to 0 degrees
- moved R7 2.11 mm to (39.4, 25.9), turned to 270 degrees
- moved R6 1.75 mm to (54.0, 26.9)
- moved R5 1.50 mm to (54.1, 29.9)
- moved C3 1.45 mm to (50.3, 32.0), turned to 0 degrees
- moved IC1 1.27 mm to (38.0, 30.9)
- moved C4 0.35 mm to (46.4, 31.5)
- moved C5 0.35 mm to (43.4, 31.4)
Connections:
- removed net N$23: IC2.SCLK, R2.1, U$2.P$13
- removed net N$32: C4.1, IC1.4, IC1.8, J1.1, LED3.A, LED4.A, R7.2
- new net N$16: U$1.P$10, U$5.P$4
- new net N$21: U$1.P$11, U$5.P$19
- new net SHIELD: J1.SH1, J1.SH2, J1.SH3, J1.SH4, J1.SH5
- net BATT+: now also R1.2, R2.2, R3.1, R7.2, U$5.P$8; no longer U$2.P$8
- net GND: now also J1.1, U$5.P$10; no longer J1.5, J1.SH1, J1.SH2, J1.SH3, J1.SH4, J1.SH5, R1.2, R2.2, R3.2, R7.1, U$2.P$10
- net N$1: now also U$5.P$3; no longer U$2.P$3
- net N$10: now also IC2.SCLK, R2.1, U$5.P$13; no longer U$1.P$10, U$2.P$4
- net N$11: now also IC2.-RST, R3.2, U$5.P$7; no longer U$1.P$11, U$2.P$19
- net N$12: now also U$5.P$15; no longer U$2.P$15
- net N$14: now also C4.1, D1.-, D2.-, IC1.4, IC1.8, J1.5, R7.1; no longer IC2.-RST, R3.1, U$2.P$7
- net N$17: now also U$5.P$9; no longer U$2.P$9
- net N$19: now also U$5.P$14; no longer U$2.P$14
- net N$2: now also U$5.P$2; no longer U$2.P$2
- net N$20: now also U$5.P$12; no longer U$2.P$12
- net N$27: now also D1.+; no longer LED4.C
- net N$29: now also D2.+; no longer LED3.C
- net N$3: now also U$5.P$1; no longer U$2.P$1
- net N$4: now also U$5.P$6; no longer U$2.P$6
- net N$5: now also U$5.P$5; no longer U$2.P$5
- net N$6: now also U$5.P$18; no longer U$2.P$18
- net N$7: now also U$5.P$20; no longer U$2.P$20
- net N$8: now also U$5.P$17; no longer U$2.P$17
- net N$9: now also U$5.P$16; no longer U$2.P$16
Routing:
- net BATT+: track 44.9 -> 101.3 mm, vias 1 -> 2
- net N$32: track 50.2 -> 0.00 mm, vias 3 -> 0
- net N$7: track 10.8 -> 56.0 mm, vias 0 -> 1
- net GND: track 175.1 -> 140.5 mm, vias 0 -> 1
- net N$10: track 2.53 -> 33.6 mm, vias 0 -> 4
- net N$21: track 0.00 -> 30.6 mm, vias 0 -> 1
- net N$23: track 29.9 -> 0.00 mm, vias 1 -> 0
- net N$8: track 13.2 -> 42.8 mm, vias 0 -> 2
- net N$16: track 0.00 -> 27.4 mm, vias 0 -> 1
- net N$9: track 12.2 -> 34.4 mm
- net N$6: track 24.8 -> 44.4 mm, vias 0 -> 4
- net N$17: track 51.0 -> 33.4 mm, vias 0 -> 2
- net N$14: track 60.3 -> 42.7 mm, vias 2 -> 1
- net SHIELD: track 0.00 -> 17.0 mm
- net N$11: track 17.8 -> 0.97 mm
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- removed copper zone on layer 1, net GND
- removed copper zone on layer 16, net GND
